Commit message: Integrate sorting_arm_gazebo world with UR10e + AG95 simulation
- Register Universal_Robots_ROS2_Description as a proper submodule
  (.gitmodules was missing; pinned commit 89bbe79 unchanged)
- sorting_arm: add mount_x/y/z xacro args (default 0, behaviour unchanged)
  and expose description_file/world_file launch args (same defaults)
- sorting_arm: fix rosdep keys ur-simulation-gz / position-controllers
- sorting_arm_gazebo: add robot pedestal and Contact system to the world,
  sorting_cell.urdf.xacro mounting the robot on it, and a single
  sorting_sim.launch.py bringing up robot, controllers, world and camera

Co-Authored-By: Claude Opus 5.5 <noreply@anthropic.com>

File: ros2_ws/src/sorting_arm/urdf/sorting_arm.urdf.xacro (robot description, xacro)
@@ -23,4 +23,8 @@
   <xacro:arg name="simulation_controllers" default="" />
   <xacro:arg name="ros_namespace" default="" />
+  <!-- robot base pose in the world; zero by default, overridden by sorting_arm_gazebo's cell -->
+  <xacro:arg name="mount_x" default="0"/>
+  <xacro:arg name="mount_y" default="0"/>
+  <xacro:arg name="mount_z" default="0"/>
   <!-- create link fixed to the "world" -->
   <link name="world" />
@@ -61,5 +65,5 @@
     force_abs_paths="true"
     >
-    <origin xyz="0 0 0" rpy="0 0 0" />          <!-- position robot in the world -->
+    <origin xyz="$(arg mount_x) $(arg mount_y) $(arg mount_z)" rpy="0 0 0" />          <!-- position robot in the world -->
   </xacro:ur_robot>
   <!-- Added end effector/tool0 here: -->
