Commit message: Align MoveIt with the Gazebo sim and fix AG95 rendering in RViz
- sorting_arm: prefix AG95 mesh URIs with file:// so RViz (resource_retriever)
  can load them; geometry unchanged. Add dh_ag95_description dependency.
- sorting_arm / sorting_arm_gazebo launches: add launch_rviz argument
  (default true) so the UR RViz can be disabled when using MoveIt's RViz.
- sorting_arm_moveit_config:
  - Use sorting_arm_gazebo/urdf/sorting_cell.urdf.xacro with the same xacro
    args as Gazebo, so MoveIt has the pedestal-mounted robot description.
  - SRDF: drop the world->base_link virtual joint (the URDF already roots at
    world with the mount) and add AG95 collision-disable pairs.
  - Add moveit_controllers.yaml mapping to
    joint_trajectory_controller/follow_joint_trajectory.
  - Add sim_moveit.launch.py (move_group + RViz on use_sim_time).
  - Enable 5.0 rad/s^2 acceleration limits (as in ur_moveit_config); time
    parameterization fails without them.
  - RViz: frame the pedestal robot, default to the arm group with the goal
    marker enabled.

File: ros2_ws/src/sorting_arm/urdf/dh_ag95_macro_for_sorting_arm.xacro (robot description, xacro)
@@ -29,5 +29,5 @@
           <origin xyz="-0.036673 0.00875 -0.098336" rpy="0 0 0" />
           <geometry>
-            <mesh filename="$(find dh_ag95_description)/meshes/visual/outer_knuckle.stl"
+            <mesh filename="file://$(find dh_ag95_description)/meshes/visual/outer_knuckle.stl"
               scale="0.001 0.001 0.001" />
           </geometry>
@@ -39,5 +39,5 @@
           <origin xyz="-0.036673 0.00875 -0.098336" rpy="0 0 0" />
           <geometry>
-            <mesh filename="$(find dh_ag95_description)/meshes/collision/outer_knuckle.stl"
+            <mesh filename="file://$(find dh_ag95_description)/meshes/collision/outer_knuckle.stl"
               scale="0.001 0.001 0.001" />
           </geometry>
@@ -60,5 +60,5 @@
           <origin xyz="-0.016 0.0254 -0.10586" rpy="0 0 0" />
           <geometry>
-            <mesh filename="$(find dh_ag95_description)/meshes/visual/inner_knuckle.stl"
+            <mesh filename="file://$(find dh_ag95_description)/meshes/visual/inner_knuckle.stl"
               scale="0.001 0.001 0.001" />
           </geometry>
@@ -70,5 +70,5 @@
           <origin xyz="-0.016 0.0254 -0.10586" rpy="0 0 0" />
           <geometry>
-            <mesh filename="$(find dh_ag95_description)/meshes/collision/inner_knuckle.stl"
+            <mesh filename="file://$(find dh_ag95_description)/meshes/collision/inner_knuckle.stl"
               scale="0.001 0.001 0.001" />
           </geometry>
@@ -91,5 +91,5 @@
           <origin xyz="-0.091673 0.00875 -0.098336" rpy="0 0 0" />
           <geometry>
-            <mesh filename="$(find dh_ag95_description)/meshes/visual/finger.stl"
+            <mesh filename="file://$(find dh_ag95_description)/meshes/visual/finger.stl"
               scale="0.001 0.001 0.001" />
           </geometry>
@@ -101,5 +101,5 @@
           <origin xyz="-0.091673 0.00875 -0.098336" rpy="0 0 0" />
           <geometry>
-            <mesh filename="$(find dh_ag95_description)/meshes/collision/finger.stl"
+            <mesh filename="file://$(find dh_ag95_description)/meshes/collision/finger.stl"
               scale="0.001 0.001 0.001" />
           </geometry>
@@ -124,5 +124,5 @@
           <origin xyz="-0.0705 -0.0 -0.12056" rpy="0 0 0" />
           <geometry>
-            <mesh filename="$(find dh_ag95_description)/meshes/visual/finger_pad.stl"
+            <mesh filename="file://$(find dh_ag95_description)/meshes/visual/finger_pad.stl"
               scale="0.001 0.001 0.001" />
           </geometry>
@@ -134,5 +134,5 @@
           <origin xyz="-0.0705 -0.0 -0.12056" rpy="0 0 0" />
           <geometry>
-            <mesh filename="$(find dh_ag95_description)/meshes/collision/finger_pad.stl"
+            <mesh filename="file://$(find dh_ag95_description)/meshes/collision/finger_pad.stl"
               scale="0.001 0.001 0.001" />
           </geometry>
@@ -215,5 +215,5 @@
         <origin xyz="0 0 0" rpy="0 0 0" />
         <geometry>
-          <mesh filename="$(find dh_ag95_description)/meshes/visual/base_link.stl"
+          <mesh filename="file://$(find dh_ag95_description)/meshes/visual/base_link.stl"
             scale="0.001 0.001 0.001" />
         </geometry>
@@ -225,5 +225,5 @@
         <origin xyz="0 0 0" rpy="0 0 0" />
         <geometry>
-          <mesh filename="$(find dh_ag95_description)/meshes/collision/base_link.stl"
+          <mesh filename="file://$(find dh_ag95_description)/meshes/collision/base_link.stl"
             scale="0.001 0.001 0.001" />
         </geometry>
@@ -245,5 +245,5 @@
         <origin xyz="0.0405 0.0143 -0.0147" rpy="0 0 0" />
         <geometry>
-          <mesh filename="$(find dh_ag95_description)/meshes/visual/gripper_body.stl"
+          <mesh filename="file://$(find dh_ag95_description)/meshes/visual/gripper_body.stl"
             scale="0.001 0.001 0.001" />
         </geometry>
@@ -255,5 +255,5 @@
         <origin xyz="0.0405 0.0143 -0.0147" rpy="0 0 0" />
         <geometry>
-          <mesh filename="$(find dh_ag95_description)/meshes/collision/gripper_body.stl"
+          <mesh filename="file://$(find dh_ag95_description)/meshes/collision/gripper_body.stl"
             scale="0.001 0.001 0.001" />
         </geometry>

Commit message: Added state machine and dummy launch file, added friction to gripper in sorting_arm

File: ros2_ws/src/sorting_arm/urdf/dh_ag95_macro_for_sorting_arm.xacro (robot description, xacro)
@@ -139,5 +139,22 @@
         </collision>
       </link>
-    </xacro:macro>
+      <!-- Gazebo friction/contact -->
+      <gazebo reference="${prefix}${fingerprefix}_finger_pad">
+        <surface>
+          <friction>
+            <ode>
+              <mu>150.0</mu>
+              <mu2>150.0</mu2>
+            </ode>
+          </friction>
+          <contact>
+            <ode>
+              <kp>1000000.0</kp>
+              <kd>1.0</kd>
+              <min_depth>0.001</min_depth>
+            </ode>
+          </contact>
+        </surface>
+      </gazebo>
     <xacro:macro name="finger_links" params="prefix fingerprefix">
       <xacro:outer_knuckle prefix="${prefix}" fingerprefix="${fingerprefix}" />

Commit message: Fix AG95 xacro: restore finger_pad macro close tag and valid friction block
The finger-pad friction edit replaced the finger_pad </xacro:macro>, so the
file no longer parsed. Restore the tag and express the friction/contact
settings with the <mu1>/<mu2>/<kp>/<kd>/<minDepth> tags that sdformat maps
onto the collision <surface> (a raw <surface> under <gazebo reference> is
ignored). Preserve the pad's fixed joint: when lumped into *_finger, sdformat
drops the pad's gazebo extension because the child name is prefixed by the
parent's.

File: ros2_ws/src/sorting_arm/urdf/dh_ag95_macro_for_sorting_arm.xacro (robot description, xacro)
@@ -139,22 +139,16 @@
         </collision>
       </link>
-      <!-- Gazebo friction/contact -->
+      <!-- Gazebo friction/contact for the pad. sdformat's URDF parser maps these
+           tags onto the link's collision <surface>; a raw <surface> block here
+           would be ignored. finger_pad_joint sets preserveFixedJoint so the pad
+           is not lumped into the finger link, which would drop these settings. -->
       <gazebo reference="${prefix}${fingerprefix}_finger_pad">
-        <surface>
-          <friction>
-            <ode>
-              <mu>150.0</mu>
-              <mu2>150.0</mu2>
-            </ode>
-          </friction>
-          <contact>
-            <ode>
-              <kp>1000000.0</kp>
-              <kd>1.0</kd>
-              <min_depth>0.001</min_depth>
-            </ode>
-          </contact>
-        </surface>
+        <mu1>150.0</mu1>
+        <mu2>150.0</mu2>
+        <kp>1000000.0</kp>
+        <kd>1.0</kd>
+        <minDepth>0.001</minDepth>
       </gazebo>
+    </xacro:macro>
     <xacro:macro name="finger_links" params="prefix fingerprefix">
       <xacro:outer_knuckle prefix="${prefix}" fingerprefix="${fingerprefix}" />
@@ -209,4 +203,7 @@
         <child link="${prefix}${fingerprefix}_finger_pad" />
       </joint>
+      <gazebo reference="${prefix}${fingerprefix}_inner_finger_pad_joint">
+        <preserveFixedJoint>true</preserveFixedJoint>
+      </gazebo>
     </xacro:macro>
     <xacro:macro name="finger_joints" params="prefix fingerprefix reflect">
